File: KiCad/SchindlerCarrierBoard_V1/SchindlerCarrierBoard_V1/03-power-tree.kicad_sch (KiCad schematic)
At the start: 81 parts, among them J300 FN9260B-6-06, J301 Molex 0039291028, U300 TPS26601 (latch-off; '600 sym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, U301 INA226AIDGSR, U302 LTC2954-1, U303 LMR33640 (5V), U304 LMR33640 (3.3V), U305 TLV62568 (1.2V), U306 TPS7A2018PDBVR, U307 ADP7142 (AD9204 AVDD)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

Commit message: Schindler 2.0: hand-wired schematic sheets (KiCad GUI)
Manual wiring pass done in KiCad: sheet 3 (power-tree), sheet 4 (HDMI
in/out), and sheet 7 (SDI) converted from net-label capture to drawn
wires + junctions (17 / 229 / 171 wires respectively). Remaining child
sheets re-saved by KiCad in native format (no logical change).
Parts:
- U300: value TPS26601 (latch-off; '600 symbol, identical pinout) -> TPS26601 (latch-off)
Connections:
- net +12V_PROT: no longer U301.8 (Vbus)
- net +3V3_A: no longer R321.1
- net EFUSE_EN: no longer U302.6 (EN/*EN)
- net PDT_RC: no longer U302.7 (PDT)
- net PWR_INT_N: no longer U302.5 (*INT)
- net PWR_KILL_N: no longer U302.8 (*KILL)
Other:
- moved on the sheet: C300, C301, C302, C303, C310, C311, C312, C313, C320, C321, C322, C323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
