File: KiCad/SchindlerCarrierBoard_V1/SchindlerCarrierBoard_V1/04-hdmi-in-out.kicad_sch (KiCad schematic)
At the start: 17 parts, among them J400 10029449-001RLF (HDMI IN), J401 10029449-001RLF (HDMI OUT), U401 TPD12S016PWR (OUT ESD/level), U402 LT8619C (HDMI RX), U403 ADV7511KSTZ (HDMI TX)

Commit message: Schindler 2.0: hand-wired schematic sheets (KiCad GUI)
Manual wiring pass done in KiCad: sheet 3 (power-tree), sheet 4 (HDMI
in/out), and sheet 7 (SDI) converted from net-label capture to drawn
wires + junctions (17 / 229 / 171 wires respectively). Remaining child
sheets re-saved by KiCad in native format (no logical change).
Parts:
- D404: value TMDS ESD <0.5pF (CLK+D0) -> TMDS ESD, TPD4E05U06DQA
- D405: value TMDS ESD <0.5pF (D1+D2) -> TMDS ESD, TPD4E05U06DQA
- D406: value DDC/HPD ESD -> DDC/HPD ESD, TPD3E001DRLR; footprint (none) -> Package_TO_SOT_SMD:SOT-553
- U401: footprint (none) -> Package_SO:TSSOP-24_4.4x7.8mm_P0.65mm
Connections:
- no-connect marks 0 -> 121
Other:
- note added: "See trace routing in TPD12S016PWR Datasheet, pg 22."
- moved on the sheet: C401, C403, C405, D404, D405, D406, J400, J401, R400, R401, R402, R403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
