File: KiCad/SchindlerCarrierBoard_V1/SchindlerCarrierBoard_V1/04-hdmi-in-out.kicad_sch (KiCad schematic)
At the start: 17 parts, among them J400 10029449-001RLF (HDMI IN), J401 10029449-001RLF (HDMI OUT), U401 TPD12S016PWR (OUT ESD/level), U402 LT8619C (HDMI RX), U403 ADV7511KSTZ (HDMI TX)

Commit message: Schindler 2.0: sheet 4 power decoupling — TPD12S016 + LT8619C
- TPD12S016 (U401): added C406 0.1 uF X7R on VCC5V (parallel to C405
  1 uF bulk); VCCA already had C403 0.1 uF.
- LT8619C (U402): full multi-supply decoupling added — 14x 0.1 uF X7R
  (one per supply pin, C407-C420) + 3x 10 uF bulk per rail (C421-C423,
  +1V8_A/+1V8_D/+3V3).
- PLL/clock jitter isolation: FB400 (+1V8_A -> PVCC18 pin 59) and FB401
  (+3V3 -> VCCA33_XTAL pin 62) ferrites, with C409/C418 0.1 uF on the
  isolated pin side (LC filter).
- ERC sheet 4: pin_not_connected 0, pin_not_driven 0; the 2
  power_pin_not_driven are the intentional HDMI +5V pins (J400/J401.18).
- bom-v1 + kicad-capture-log (sec 26/27) reconciled.

Co-Authored-By: Claude Opus 4.8 (1M context) <noreply@anthropic.com>
Parts:
- added C406: 0.1uF (U401 VCC5V HF, X7R), symbol Device:C
- added C407: 0.1uF (U402 CT_HPD), symbol Device:C
- added C408: 0.1uF (U402 VCCA18), symbol Device:C
- added C409: 0.1uF (U402 PVCC18), symbol Device:C
- added C410, C411, C412: 0.1uF (U402 VDD18), symbol Device:C
- added C413: 0.1uF (U402 VCCA33), symbol Device:C
- added C414, C415: 0.1uF (U402 VCC33), symbol Device:C
- added C416, C417: 0.1uF (U402 VCC33_TTL), symbol Device:C
- added C418: 0.1uF (U402 VCCA33_XTAL), symbol Device:C
- added C419, C420: 0.1uF (U402 VTERM), symbol Device:C
- added C421: 10uF (U402, +1V8_A), symbol Device:C
- added C422: 10uF (U402, +1V8_D), symbol Device:C
- added C423: 10uF (U402, +3V3), symbol Device:C
- added FB400, FB401: U402, 600 Ω @ 100 MHz, symbol Device:FerriteBead
Connections:
- net +1V8_A: now also C407.1, C408.1, C421.1, FB400.2; no longer U402.59 (PVCC18)
- net +1V8_D: now also C410.1, C411.1, C412.1, C422.1
- net +3V3: now also C413.1, C414.1, C415.1, C416.1, C417.1, C419.1, C420.1, C423.1, FB401.1; no longer U402.62 (VCCA33_XTAL)
- net +5V: now also C406.1
- net GND: now also C406.2, C407.2, C408.2, C409.2, C410.2, C411.2, C412.2, C413.2, C414.2, C415.2, C416.2, C417.2, C418.2, C419.2, C420.2, C421.2, C422.2, C423.2
- new net: C409.1, FB400.1, U402.59 (PVCC18)
- new net: C418.1, FB401.2, U402.62 (VCCA33_XTAL)
Other:
- moved on the sheet: C401, C403, C405, D404, D405, D406, J400, R404, R405, U401

Commit message: Schindler 2.0: checkpoint — decoupling + functional audit, pre-edit save
Saves current carrier schematic state (all 12 sheets, KiCad re-saves) and
project docs before starting the decoupling/functional-fix wiring pass.

- docs/decoupling-audit.md: full per-chip decoupling audit (EXISTS /
  DATASHEET WANTS / PROPOSED ADDS) + "Functional fixes" section
  (COMP/PWRDWN*/VREG_VOUT floating, Y900 load caps; clocks verified
  present). ~91 proposed caps + ferrites; report-only, nothing placed.
- Other docs (bom-v1, refdes-map, spec, part-lock, etc.) synced.

No wiring changes — proposals await gate. Reference binaries (datasheet
JPGs/PDF, Manufacturing/) intentionally left untracked.

Co-Authored-By: Claude Opus 4.8 (1M context) <noreply@anthropic.com>
Parts:
- C401, C403, C405, C406, C407, C408, C409, C410, C411, C412, C413, C414, C415, C416, C417, C418, C419, C420, C421, C422, C423: footprint (none) -> Capacitor_SMD:C_0805_2012Metric
- R400, R401, R402, R403, R404, R405: footprint (none) -> Resistor_SMD:R_0805_2012Metric
Changed lines of the file:
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@@
 			)
 		)
-		(property "Footprint" ""
+		(property "Footprint" "Capacitor_SMD:C_0805_2012Metric"
 			(at 218.44 309.88 0)
 			(hide yes)
@@
 			)
 		)
-		(property "Footprint" ""
+		(property "Footprint" "Resistor_SMD:R_0805_2012Metric"
 			(at 290.83 156.21 0)
 			(hide yes)
@@
 			)
 		)
-		(property "Footprint" ""
+		(property "Footprint" "Resistor_SMD:R_0805_2012Metric"
 			(at 445.77 139.7 0)
 			(hide yes)
@@
 			)
 		)
-		(property "Footprint" ""
+		(property "Footprint" "Resistor_SMD:R_0805_2012Metric"
 			(at 445.77 149.86 0)
 			(hide yes)
@@
 			)
 		)
-		(property "Footprint" ""
+		(property "Footprint" "Capacitor_SMD:C_0805_2012Metric"
 			(at 464.82 212.09 0)
 			(hide yes)
@@
 			)
 		)
-		(property "Footprint" ""
+		(property "Footprint" "Capacitor_SMD:C_0805_2012Metric"
 			(at 181.61 334.01 0)
 			(hide yes)
@@
 			)
 		)
-		(property "Footprint" ""
+		(property "Footprint" "Capacitor_SMD:C_0805_2012Metric"
 			(at 218.44 284.48 0)
 			(hide yes)
@@
 			)
 		)
-		(property "Footprint" ""
+		(property "Footprint" "Capacitor_SMD:C_0805_2012Metric"
 			(at 486.41 158.75 0)
 			(hide yes)
@@
 			)
 		)
-		(property "Footprint" ""
+		(property "Footprint" "Capacitor_SMD:C_0805_2012Metric"
 			(at 260.35 297.18 0)
 			(hide yes)
@@
 			)
 		)
-		(property "Footprint" ""
+		(property "Footprint" "Resistor_SMD:R_0805_2012Metric"
 			(at 290.83 147.32 0)
 			(hide yes)
@@
 			)
 		)
-		(property "Footprint" ""
+		(property "Footprint" "Resistor_SMD:R_0805_2012Metric"
 			(at 299.72 227.33 0)
 			(hide yes)
@@
 			)
 		)
-		(property "Footprint" ""
+		(property "Footprint" "Capacitor_SMD:C_0805_2012Metric"
 			(at 302.26 297.18 0)
 			(hide yes)
@@
 			)
 		)
-		(property "Footprint" ""
+		(property "Footprint" "Capacitor_SMD:C_0805_2012Metric"
 			(at 173.99 297.18 0)
 			(hide yes)
@@
 			)
 		)
-		(property "Footprint" ""
+		(property "Footprint" "Capacitor_SMD:C_0805_2012Metric"
 			(at 173.99 284.48 0)
 			(hide yes)
@@
 			)
 		)
-		(property "Footprint" ""
+		(property "Footprint" "Capacitor_SMD:C_0805_2012Metric"
 			(at 260.35 309.88 0)
 			(hide yes)
@@
 			)
 		)
-		(property "Footprint" ""
+		(property "Footprint" "Capacitor_SMD:C_0805_2012Metric"
 			(at 260.35 271.78 0)
 			(hide yes)
@@
 			)
 		)
-		(property "Footprint" ""
+		(property "Footprint" "Resistor_SMD:R_0805_2012Metric"
 			(at 299.72 236.22 0)
 			(hide yes)
@@
 			)
 		)
-		(property "Footprint" ""
+		(property "Footprint" "Capacitor_SMD:C_0805_2012Metric"
 			(at 464.82 223.52 0)
 			(hide yes)
@@
 			)
 		)
-		(property "Footprint" ""
+		(property "Footprint" "Capacitor_SMD:C_0805_2012Metric"
 			(at 218.44 297.18 0)
 			(hide yes)
@@
 			)
 		)
-		(property "Footprint" ""
+		(property "Footprint" "Capacitor_SMD:C_0805_2012Metric"
 			(at 175.26 271.78 0)
 			(hide yes)
@@
 			)
 		)
-		(property "Footprint" ""
+		(property "Footprint" "Capacitor_SMD:C_0805_2012Metric"
 			(at 173.99 309.88 0)
 			(hide yes)
@@
 			)
 		)
-		(property "Footprint" ""
+		(property "Footprint" "Capacitor_SMD:C_0805_2012Metric"
 			(at 302.26 309.88 0)
 			(hide yes)
@@
 			)
 		)
-		(property "Footprint" ""
+		(property "Footprint" "Capacitor_SMD:C_0805_2012Metric"
 			(at 464.82 234.95 0)
 			(hide yes)
@@
 			)
 		)
-		(property "Footprint" ""
+		(property "Footprint" "Capacitor_SMD:C_0805_2012Metric"
 			(at 242.57 334.01 0)
 			(hide yes)
@@
 			)
 		)
-		(property "Footprint" ""
+		(property "Footprint" "Capacitor_SMD:C_0805_2012Metric"
 			(at 218.44 271.78 0)
 			(hide yes)
@@
 			)
 		)
-		(property "Footprint" ""
+		(property "Footprint" "Capacitor_SMD:C_0805_2012Metric"
 			(at 260.35 284.48 0)
 			(hide yes)
@@
 			)
 		)
-		(property "Footprint" ""
+		(property "Footprint" "Capacitor_SMD:C_0805_2012Metric"
 			(at 213.36 334.01 0)
 			(hide yes)

Commit message: Schindler carrier: ADV7511 R_EXT/AVDD fix + symbol relabel; 116 PL nets wired; connector/riser decisions
- U403 ADV7511: add R406 (887R 1%) pin28 R_EXT->GND; wire pin29 AVDD->+1V8_A (match 34/41).
  Sheet-4 ERC pin_not_connected 2->0. Fixes missing TMDS bias ref + unpowered AVDD
  (would-not-work HDMI-out bug, caught pre-fab).
- JustinLibrary ADV7511KSTZ symbol relabel: pin2 SYNC->VSYNC, 28 EXT->R_EXT, 29 R_EXT->AVDD
  (cosmetic; connectivity is by pin number). [NOTE: JustinLibrary is unversioned/external — not in this repo; see report.]
- Pin-lock: 116 PL nets wired; ERC unconnected 899->668; schindler_plio.xdc + pin-lock-assignment.md.
- Connector domain + analog I/O riser decided (connector-domain.md); riser-mezzanine-plan.md rev2
  (gated proposal, not implemented).
- bom-v1 (R406), refdes-map (R406 + symbol-mislabel note), changelog.

Deferred to next commit (kept out so this push stays honest): eeschema Update Symbols from
Library on U403 (display refresh); netlist regen; HDMI +5V power_pin_not_driven x2 (J400/J401.18)
verification; riser stays gated.

Co-Authored-By: Claude Opus 4.8 (1M context) <noreply@anthropic.com>
Parts:
- added C424, C425, C426, C427, C428: 0.1uF (U403 DVDD), Capacitor_SMD:C_0805_2012Metric, symbol Device:C
- added C429, C430: 0.1uF (U403 AVDD), Capacitor_SMD:C_0805_2012Metric, symbol Device:C
- added C433: 10uF (U403 DVDD/AVDD bulk), Capacitor_SMD:C_0805_2012Metric, symbol Device:C
- added R406: 887 1% (U403 R_EXT bias), symbol Device:R
Connections:
- net +1V8_A: now also U403.29 (R_EXT), C424.1, C425.1, C426.1, C427.1, C428.1, C429.1, C430.1, C433.1
- net GND: now also C424.2, C425.2, C426.2, C427.2, C428.2, C429.2, C430.2, C433.2, R406.2
- net HDMITX_VS: now reaches U403.2 (SYNC)
- net U403_REXT: now reaches U403.28 (EXT)
- net U403_REXT: now also R406.1
- net HDMITX_PCLK: now reaches U403.79 (CLK)
- net HDMITX_D15: now reaches U403.81 (D15)
- net HDMITX_D14: now reaches U403.82 (D14)
- net HDMITX_D13: now reaches U403.83 (D13)
- net HDMITX_D12: now reaches U403.84 (D12)
- net HDMITX_D11: now reaches U403.85 (D11)
- net HDMITX_D10: now reaches U403.86 (D10)
- net HDMITX_D9: now reaches U403.87 (D9)
- net HDMITX_D8: now reaches U403.88 (D8)
- net HDMITX_D7: now reaches U403.89 (D7)
- net HDMITX_D6: now reaches U403.90 (D6)
- net HDMITX_D5: now reaches U403.91 (D5)
- net HDMITX_D4: now reaches U403.92 (D4)
- net HDMITX_D3: now reaches U403.93 (D3)
- net HDMITX_D2: now reaches U403.94 (D2)
- net HDMITX_D1: now reaches U403.95 (D1)
- net HDMITX_D0: now reaches U403.96 (D0)
- net HDMITX_DE: now reaches U403.97 (DE)
- net HDMITX_HS: now reaches U403.98 (HSYNC)
- net HDMIRX_D15: now reaches U402.37 (D15_TC3+)
- net HDMIRX_D14: now reaches U402.38 (D14_TC3-)
- net HDMIRX_D13: now reaches U402.39 (D13_TCC+)
- net HDMIRX_D12: now reaches U402.40 (D12_TCC-)
- net HDMIRX_D11: now reaches U402.41 (D11_TC2+)
- net HDMIRX_D10: now reaches U402.42 (D10_TC2-)
- net HDMIRX_D9: now reaches U402.43 (D9_TC1+)
- net HDMIRX_D8: now reaches U402.44 (D8_TC1-)
- net HDMIRX_D7: now reaches U402.45 (D7_TC0+)
- net HDMIRX_D6: now reaches U402.46 (D6_TC0-)
- net HDMIRX_D5: now reaches U402.47 (D5)
- net HDMIRX_D4: now reaches U402.48 (D4)
- net HDMIRX_D3: now reaches U402.49 (D3)
- net HDMIRX_D2: now reaches U402.50 (D2)
- net HDMIRX_D1: now reaches U402.51 (D1)
- net HDMIRX_D0: now reaches U402.52 (D0)
- net HDMIRX_DE: now reaches U402.53 (DE)
- net HDMIRX_HS: now reaches U402.54 (HS)
- net HDMIRX_VS: now reaches U402.55 (VS)
- net HDMIRX_PCLK: now reaches U402.56 (PCLK)
- no-connect marks 121 -> 81
Other:
- moved on the sheet: C401, C403, C405, C406, J401, R402, R403, U401
