File: KiCad/SchindlerCarrierBoard_V1/SchindlerCarrierBoard_V1/07-sdi.kicad_sch (KiCad schematic)
At the start: 44 parts, among them J700 73101-0120 (SDI IN), J701 73101-0120 (SDI OUT 1), J702 73101-0120 (SDI IN LOOP), J703 73101-0120 (SDI OUT 2 mirror), U700 GS3470 (SDI RX), U701 GS2962 (SDI TX), U702 LMH0302-class 3G-SDI loop dri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, Y700 27MHz 9pF-CL (GS3470 ref; con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

Commit message: Schindler 2.0: hand-wired schematic sheets (KiCad GUI)
Manual wiring pass done in KiCad: sheet 3 (power-tree), sheet 4 (HDMI
in/out), and sheet 7 (SDI) converted from net-label capture to drawn
wires + junctions (17 / 229 / 171 wires respectively). Remaining child
sheets re-saved by KiCad in native format (no logical change).
Parts:
- C704: value 4.7uF (SDI OUT AC-couple) -> 4.7uF (AC-couple)
- L700: value 5.6nH (SDO series, ||75; RF wideband, SRF>3G, verify MPN) -> 5.6nH
- U702: value LMH0302-class 3G-SDI loop driver -> 3G-SDI loop driver, LMH0302SQE/NOPB; footprint (none) -> Package_DFN_QFN:WQFN-16-1EP_4x4mm_P0.5mm_EP2.6x2.6mm
Connections:
- net GND: now also C701.1; no longer C701.2
- net GS3470_nDDI0: now also C701.2; no longer C701.1
- no-connect marks 0 -> 106
Other:
- moved on the sheet: C700, C701, C702, C703, C704, C705, C706, C707, C708, C709, C710, C711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
