File: KiCad/SchindlerCarrierBoard_V1/SchindlerCarrierBoard_V1/07-sdi.kicad_sch (KiCad schematic)
At the start: 44 parts, among them J700 73101-0120 (SDI IN), J701 73101-0120 (SDI OUT 1), J702 73101-0120 (SDI IN LOOP), J703 73101-0120 (SDI OUT 2 mirror), U700 GS3470 (SDI RX), U701 GS2962 (SDI TX), U702 3G-SDI loop driver, LMH0302SQ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, Y700 27MHz 9pF-CL (GS3470 ref; con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

Commit message: Schindler 2.0: checkpoint — decoupling + functional audit, pre-edit save
Saves current carrier schematic state (all 12 sheets, KiCad re-saves) and
project docs before starting the decoupling/functional-fix wiring pass.

- docs/decoupling-audit.md: full per-chip decoupling audit (EXISTS /
  DATASHEET WANTS / PROPOSED ADDS) + "Functional fixes" section
  (COMP/PWRDWN*/VREG_VOUT floating, Y900 load caps; clocks verified
  present). ~91 proposed caps + ferrites; report-only, nothing placed.
- Other docs (bom-v1, refdes-map, spec, part-lock, etc.) synced.

No wiring changes — proposals await gate. Reference binaries (datasheet
JPGs/PDF, Manufacturing/) intentionally left untracked.

Co-Authored-By: Claude Opus 4.8 (1M context) <noreply@anthropic.com>
Parts:
- C700, C701, C702, C703, C704, C705, C706, C707, C708, C709, C710, C711, C712, C713, C714, C715, C720, C721, C722: footprint (none) -> Capacitor_SMD:C_0805_2012Metric
- R704, R705, R720, R722, R723, R725, R726, R727: footprint (none) -> Resistor_SMD:R_0805_2012Metric
Changed lines of the file:
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@@
 			)
 		)
-		(property "Footprint" ""
+		(property "Footprint" "Resistor_SMD:R_0805_2012Metric"
 			(at 377.19 241.3 0)
 			(hide yes)
@@
 			)
 		)
-		(property "Footprint" ""
+		(property "Footprint" "Capacitor_SMD:C_0805_2012Metric"
 			(at 363.22 161.29 0)
 			(hide yes)
@@
 			)
 		)
-		(property "Footprint" ""
+		(property "Footprint" "Capacitor_SMD:C_0805_2012Metric"
 			(at 382.27 196.85 0)
 			(hide yes)
@@
 			)
 		)
-		(property "Footprint" ""
+		(property "Footprint" "Resistor_SMD:R_0805_2012Metric"
 			(at 261.62 146.05 0)
 			(hide yes)
@@
 			)
 		)
-		(property "Footprint" ""
+		(property "Footprint" "Capacitor_SMD:C_0805_2012Metric"
 			(at 127 213.36 0)
 			(hide yes)
@@
 			)
 		)
-		(property "Footprint" ""
+		(property "Footprint" "Resistor_SMD:R_0805_2012Metric"
 			(at 392.43 314.96 0)
 			(hide yes)
@@
 			)
 		)
-		(property "Footprint" ""
+		(property "Footprint" "Capacitor_SMD:C_0805_2012Metric"
 			(at 347.98 241.3 0)
 			(hide yes)
@@
 			)
 		)
-		(property "Footprint" ""
+		(property "Footprint" "Resistor_SMD:R_0805_2012Metric"
 			(at 115.57 135.89 0)
 			(hide yes)
@@
 			)
 		)
-		(property "Footprint" ""
+		(property "Footprint" "Resistor_SMD:R_0805_2012Metric"
 			(at 499.11 255.27 0)
 			(hide yes)
@@
 			)
 		)
-		(property "Footprint" ""
+		(property "Footprint" "Capacitor_SMD:C_0805_2012Metric"
 			(at 165.1 119.38 0)
 			(hide yes)
@@
 			)
 		)
-		(property "Footprint" ""
+		(property "Footprint" "Capacitor_SMD:C_0805_2012Metric"
 			(at 129.54 241.3 0)
 			(hide yes)
@@
 			)
 		)
-		(property "Footprint" ""
+		(property "Footprint" "Capacitor_SMD:C_0805_2012Metric"
 			(at 168.91 142.24 0)
 			(hide yes)
@@
 			)
 		)
-		(property "Footprint" ""
+		(property "Footprint" "Capacitor_SMD:C_0805_2012Metric"
 			(at 99.06 171.45 0)
 			(hide yes)
@@
 			)
 		)
-		(property "Footprint" ""
+		(property "Footprint" "Capacitor_SMD:C_0805_2012Metric"
 			(at 129.54 255.27 0)
 			(hide yes)
@@
 			)
 		)
-		(property "Footprint" ""
+		(property "Footprint" "Capacitor_SMD:C_0805_2012Metric"
 			(at 261.62 132.08 0)
 			(hide yes)
@@
 			)
 		)
-		(property "Footprint" ""
+		(property "Footprint" "Capacitor_SMD:C_0805_2012Metric"
 			(at 424.18 300.99 0)
 			(hide yes)
@@
 			)
 		)
-		(property "Footprint" ""
+		(property "Footprint" "Capacitor_SMD:C_0805_2012Metric"
 			(at 392.43 326.39 0)
 			(hide yes)
@@
 			)
 		)
-		(property "Footprint" ""
+		(property "Footprint" "Capacitor_SMD:C_0805_2012Metric"
 			(at 424.18 289.56 0)
 			(hide yes)
@@
 			)
 		)
-		(property "Footprint" ""
+		(property "Footprint" "Capacitor_SMD:C_0805_2012Metric"
 			(at 250.19 207.01 0)
 			(hide yes)
@@
 			)
 		)
-		(property "Footprint" ""
+		(property "Footprint" "Resistor_SMD:R_0805_2012Metric"
 			(at 227.33 146.05 0)
 			(hide yes)
@@
 			)
 		)
-		(property "Footprint" ""
+		(property "Footprint" "Resistor_SMD:R_0805_2012Metric"
 			(at 392.43 283.21 0)
 			(hide yes)
@@
 			)
 		)
-		(property "Footprint" ""
+		(property "Footprint" "Resistor_SMD:R_0805_2012Metric"
 			(at 392.43 292.1 0)
 			(hide yes)
@@
 			)
 		)
-		(property "Footprint" ""
+		(property "Footprint" "Capacitor_SMD:C_0805_2012Metric"
 			(at 227.33 129.54 0)
 			(hide yes)
@@
 			)
 		)
-		(property "Footprint" ""
+		(property "Footprint" "Capacitor_SMD:C_0805_2012Metric"
 			(at 290.83 199.39 0)
 			(hide yes)
@@
 			)
 		)
-		(property "Footprint" ""
+		(property "Footprint" "Capacitor_SMD:C_0805_2012Metric"
 			(at 382.27 208.28 0)
 			(hide yes)
@@
 			)
 		)
-		(property "Footprint" ""
+		(property "Footprint" "Capacitor_SMD:C_0805_2012Metric"
 			(at 99.06 160.02 0)
 			(hide yes)
@@
 			)
 		)
-		(property "Footprint" ""
+		(property "Footprint" "Capacitor_SMD:C_0805_2012Metric"
 			(at 363.22 179.07 0)
 			(hide yes)

Commit message: Schindler carrier: ADV7511 R_EXT/AVDD fix + symbol relabel; 116 PL nets wired; connector/riser decisions
- U403 ADV7511: add R406 (887R 1%) pin28 R_EXT->GND; wire pin29 AVDD->+1V8_A (match 34/41).
  Sheet-4 ERC pin_not_connected 2->0. Fixes missing TMDS bias ref + unpowered AVDD
  (would-not-work HDMI-out bug, caught pre-fab).
- JustinLibrary ADV7511KSTZ symbol relabel: pin2 SYNC->VSYNC, 28 EXT->R_EXT, 29 R_EXT->AVDD
  (cosmetic; connectivity is by pin number). [NOTE: JustinLibrary is unversioned/external — not in this repo; see report.]
- Pin-lock: 116 PL nets wired; ERC unconnected 899->668; schindler_plio.xdc + pin-lock-assignment.md.
- Connector domain + analog I/O riser decided (connector-domain.md); riser-mezzanine-plan.md rev2
  (gated proposal, not implemented).
- bom-v1 (R406), refdes-map (R406 + symbol-mislabel note), changelog.

Deferred to next commit (kept out so this push stays honest): eeschema Update Symbols from
Library on U403 (display refresh); netlist regen; HDMI +5V power_pin_not_driven x2 (J400/J401.18)
verification; riser stays gated.

Co-Authored-By: Claude Opus 4.8 (1M context) <noreply@anthropic.com>
Parts:
- removed C703: 4.7uF (~DDO AC-gnd), Capacitor_SMD:C_0805_2012Metric, symbol Device:C
- added C716: 1uF (+1V2 bulk), Capacitor_SMD:C_0805_2012Metric, symbol Device:C
- added C717: 10uF (+1V2 bulk), Capacitor_SMD:C_0805_2012Metric, symbol Device:C
- added C723, C724, C744, C745, C750, C751: 0.1uF (U700 CORE_VDD), Capacitor_SMD:C_0805_2012Metric, symbol Device:C
- added C725, C726, C747: 0.1uF (U700 PLL_VDD), Capacitor_SMD:C_0805_2012Metric, symbol Device:C
- added C727, C748: 0.1uF (U700 VCO_VDD), Capacitor_SMD:C_0805_2012Metric, symbol Device:C
- added C728, C729: 0.1uF (U700 DDI0_VDD), Capacitor_SMD:C_0805_2012Metric, symbol Device:C
- added C730: 0.1uF (U700 DDO_VDD), Capacitor_SMD:C_0805_2012Metric, symbol Device:C
- added C731, C732, C742, C743: 0.1uF (U700 IO_VDD), Capacitor_SMD:C_0805_2012Metric, symbol Device:C
- added C733, C734: 0.1uF (U701 CORE_VDD), Capacitor_SMD:C_0805_2012Metric, symbol Device:C
- added C735, C741: 0.1uF (U701 PLL_VDD), Capacitor_SMD:C_0805_2012Metric, symbol Device:C
- added C736: 0.1uF (U701 VCO_VDD), Capacitor_SMD:C_0805_2012Metric, symbol Device:C
- added C737, C740: 0.1uF (U701 IO_VDD), Capacitor_SMD:C_0805_2012Metric, symbol Device:C
- added C738: 0.1uF (U701 A_VDD), Capacitor_SMD:C_0805_2012Metric, symbol Device:C
- added C739: 0.1uF (U701 CD_VDD), Capacitor_SMD:C_0805_2012Metric, symbol Device:C
- added C746, C749: 0.1uF (U700 DDI1_VDD), Capacitor_SMD:C_0805_2012Metric, symbol Device:C
Connections:
- net +1V2: now also C716.1, C717.1, C723.1, C724.1, C733.1, C734.1, C744.1, C745.1, C750.1, C751.1
- net +1V2_A: now also C725.1, C726.1, C727.1, C728.1, C729.1, C735.1, C736.2, C741.1, C746.1, C747.1, C748.1, C749.1
- net +1V8_D: now also C731.1, C732.1, C737.1, C740.1, C742.1, C743.1
- net +3V3_A: now also C738.1
- net +3V3_SDIDRV: now also C739.1
- net GND: now also C716.2, C717.2, C723.2, C724.2, C725.2, C726.2, C727.2, C728.2, C729.2, C730.2, C731.2, C732.2, C733.2, C734.2, C735.2, C736.1, C737.2, C738.2, C739.2, C740.2, C741.2, C742.2, C743.2, C744.2, C745.2, C746.2, C747.2, C748.2, C749.2, C750.2, C751.2
- net SDI_DDO_VDD: now also C730.1
- net SDIRX_PCLK: now reaches U700.A8 (PCLK)
- net SDIRX_D9: now reaches U700.F10 (DOUT9)
- net SDIRX_D8: now reaches U700.F9 (DOUT8)
- net SDIRX_D7: now reaches U700.H10 (DOUT7)
- net SDIRX_D6: now reaches U700.H9 (DOUT6)
- net SDIRX_D5: now reaches U700.J10 (DOUT5)
- net SDIRX_D1: now reaches U700.J8 (DOUT1)
- net SDIRX_D4: now reaches U700.J9 (DOUT4)
- net SDIRX_D3: now reaches U700.K10 (DOUT3)
- net SDIRX_D0: now reaches U700.K8 (DOUT0)
- net SDIRX_D2: now reaches U700.K9 (DOUT2)
- net SDITX_PCLK: now reaches U701.B4 (PCLK)
- net SDITX_D9: now reaches U701.F1 (DIN9)
- net SDITX_D8: now reaches U701.F2 (DIN8)
- net SDITX_D7: now reaches U701.H1 (DIN7)
- net SDITX_D6: now reaches U701.H2 (DIN6)
- net SDITX_D5: now reaches U701.J1 (DIN5)
- net SDITX_D4: now reaches U701.J2 (DIN4)
- net SDITX_D1: now reaches U701.J3 (DIN1)
- net SDITX_D3: now reaches U701.K1 (DIN3)
- net SDITX_D2: now reaches U701.K2 (DIN2)
- net SDITX_D0: now reaches U701.K3 (DIN0)
- no-connect marks 106 -> 84
Other:
- moved on the sheet: C702, C706, C707, C708, C709, C710, C711, C712, C713, C714, C715, C720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
