File: KiCad/SchindlerCarrierBoard_V1/SchindlerCarrierBoard_V1/02-te0720-som-backbone.kicad_sch (KiCad schematic)
At the start: 13 parts, among them J200 Samtec LSHM-150 (JM1), J201 Samtec LSHM-150 (JM2), J202 Samtec LSHM-130 (JM3)

Commit message: Schindler carrier: ADV7511 R_EXT/AVDD fix + symbol relabel; 116 PL nets wired; connector/riser decisions
- U403 ADV7511: add R406 (887R 1%) pin28 R_EXT->GND; wire pin29 AVDD->+1V8_A (match 34/41).
  Sheet-4 ERC pin_not_connected 2->0. Fixes missing TMDS bias ref + unpowered AVDD
  (would-not-work HDMI-out bug, caught pre-fab).
- JustinLibrary ADV7511KSTZ symbol relabel: pin2 SYNC->VSYNC, 28 EXT->R_EXT, 29 R_EXT->AVDD
  (cosmetic; connectivity is by pin number). [NOTE: JustinLibrary is unversioned/external — not in this repo; see report.]
- Pin-lock: 116 PL nets wired; ERC unconnected 899->668; schindler_plio.xdc + pin-lock-assignment.md.
- Connector domain + analog I/O riser decided (connector-domain.md); riser-mezzanine-plan.md rev2
  (gated proposal, not implemented).
- bom-v1 (R406), refdes-map (R406 + symbol-mislabel note), changelog.

Deferred to next commit (kept out so this push stays honest): eeschema Update Symbols from
Library on U403 (display refresh); netlist regen; HDMI +5V power_pin_not_driven x2 (J400/J401.18)
verification; riser stays gated.

Co-Authored-By: Claude Opus 4.8 (1M context) <noreply@anthropic.com>
Parts:
- added C200, C201: 47uF (TE0720 +5V bulk, verify-Trenz), Capacitor_SMD:C_0805_2012Metric, symbol Device:C
- added C202, C203: 22uF (TE0720 +3V3 bulk, verify-Trenz), Capacitor_SMD:C_0805_2012Metric, symbol Device:C
- added C204: 10uF (TE0720 +1V8_D bulk, verify-Trenz), Capacitor_SMD:C_0805_2012Metric, symbol Device:C
- added C205, C206, C207: 0.1uF (TE0720 +5V), Capacitor_SMD:C_0805_2012Metric, symbol Device:C
- added C208, C209, C210, C211: 0.1uF (TE0720 +3V3), Capacitor_SMD:C_0805_2012Metric, symbol Device:C
- added C212: 0.1uF (TE0720 +1V8_D), Capacitor_SMD:C_0805_2012Metric, symbol Device:C
- added C213: 1uF (J200.28 EN1 soft-start), symbol Device:C
- added R213: 10k (J200.28 EN1 pull-up), symbol Device:R
- added R214: 0R (J200.7 NOSEQ -> GND), symbol Device:R
- added R215: 10k (J200.30 PGOOD pull-up), symbol Device:R
- added R216: 10k (J200.32 MODE pull-up), symbol Device:R
- added R217: 10k (J200.89 JTAGMODE pull-down), symbol Device:R
- added R218: 10k (J201.18 RESIN pull-up), symbol Device:R
Connections:
- net +1V8_D: now also C204.1, C212.1
- net +3V3: now also C202.1, C203.1, C208.1, C209.1, C210.1, C211.1, R213.2, R215.2, R216.2, R218.2; no longer J200.7 (P7)
- net +5V: now also C200.1, C201.1, C205.1, C206.1, C207.1
- net SDIRX_D3: now reaches J202.10 (Pin_10)
- net SDIRX_D4: now reaches J202.13 (Pin_13)
- net SDIRX_D5: now reaches J202.14 (Pin_14)
- net SDIRX_D6: now reaches J202.15 (Pin_15)
- net SDIRX_D7: now reaches J202.16 (Pin_16)
- net SDIRX_D8: now reaches J202.19 (Pin_19)
- net SDIRX_D9: now reaches J202.20 (Pin_20)
- net SDITX_D0: now reaches J202.21 (Pin_21)
- net SDITX_D1: now reaches J202.22 (Pin_22)
- net SDITX_D2: now reaches J202.25 (Pin_25)
- net SDITX_D3: now reaches J202.26 (Pin_26)
- net SDITX_D4: now reaches J202.27 (Pin_27)
- net SDITX_D5: now reaches J202.28 (Pin_28)
- net SDIRX_PCLK: now reaches J202.31 (Pin_31)
- net SDITX_PCLK: now reaches J202.32 (Pin_32)
- net SDITX_D6: now reaches J202.33 (Pin_33)
- net SDITX_D7: now reaches J202.34 (Pin_34)
- net SDITX_D8: now reaches J202.37 (Pin_37)
- net SDITX_D9: now reaches J202.38 (Pin_38)
- net SDIRX_D0: now reaches J202.7 (Pin_7)
- net SDIRX_D1: now reaches J202.8 (Pin_8)
- net SDIRX_D2: now reaches J202.9 (Pin_9)
- net SOM_EN1: now reaches J200.28 (P28)
- net SOM_EN1: now also C213.1, R213.1
- net SOM_PGOOD: now reaches J200.30 (P30)
- net SOM_PGOOD: now also R215.1
- net ADV7280_P0: now reaches J200.31 (P31)
- net BOOT_MODE_SEL: now reaches J200.32 (P32)
- net BOOT_MODE_SEL: now also R216.1
- net ADV7280_P1: now reaches J200.33 (P33)
- net ADV7280_P2: now reaches J200.35 (P35)
- net ADV7280_P3: now reaches J200.36 (P36)
- net ADV7280_P4: now reaches J200.37 (P37)
- net ADV7280_P5: now reaches J200.38 (P38)
- net ADV7280_P6: now reaches J200.40 (P40)
- net ADV7280_P7: now reaches J200.41 (P41)
- net HDMIRX_D0: now reaches J200.42 (P42)
- net HDMIRX_D1: now reaches J200.43 (P43)
- net HDMIRX_D2: now reaches J200.45 (P45)
- net HDMIRX_D3: now reaches J200.46 (P46)
- net HDMIRX_D4: now reaches J200.47 (P47)
- net HDMIRX_D5: now reaches J200.48 (P48)
- net HDMIRX_D6: now reaches J200.49 (P49)
- net HDMIRX_D7: now reaches J200.50 (P50)
- net HDMIRX_D8: now reaches J200.51 (P51)
- net HDMIRX_D9: now reaches J200.52 (P52)
- net HDMIRX_D10: now reaches J200.55 (P55)
- net HDMIRX_D11: now reaches J200.56 (P56)
- net HDMIRX_D12: now reaches J200.57 (P57)
- net HDMIRX_D13: now reaches J200.58 (P58)
- net HDMIRX_D14: now reaches J200.59 (P59)
- net HDMIRX_D15: now reaches J200.60 (P60)
- net HDMIRX_PCLK: now reaches J200.61 (P61)
- net HDMIRX_DE: now reaches J200.62 (P62)
- net HDMIRX_HS: now reaches J200.65 (P65)
- net HDMIRX_VS: now reaches J200.66 (P66)
- net SYNC1_DAC_CLK: now reaches J200.67 (P67)
- net SYNC1_DAC_DB0: now reaches J200.68 (P68)
- net SYNC1_DAC_DB1: now reaches J200.69 (P69)
- net SYNC1_DAC_DB2: now reaches J200.70 (P70)
- net SYNC1_DAC_DB3: now reaches J200.71 (P71)
- net SYNC1_DAC_DB4: now reaches J200.72 (P72)
- net SYNC1_DAC_DB5: now reaches J200.75 (P75)
- net SYNC1_DAC_DB6: now reaches J200.76 (P76)
- net ADV7280_LLC: now reaches J200.77 (P77)
- net SYNC1_DAC_DB7: now reaches J200.78 (P78)
- net SYNC1_DAC_DB8: now reaches J200.80 (P80)
- net SYNC1_DAC_DB9: now reaches J200.81 (P81)
- net SYNC1_DAC_DB10: now reaches J200.82 (P82)
- net SYNC1_DAC_DB11: now reaches J200.83 (P83)
- net SOM_JTAGMODE: now reaches J200.89 (P89)
- net SOM_JTAGMODE: now also R217.1
- net GENADC_D0: now reaches J201.11 (P11)
- net GENADC_D1: now reaches J201.13 (P13)
- net GENADC_D2: now reaches J201.14 (P14)
- net GENADC_D3: now reaches J201.15 (P15)
- net GENADC_D4: now reaches J201.16 (P16)
- net GENADC_D5: now reaches J201.17 (P17)
- net SOM_RESET_N: now reaches J201.18 (P18)
- net SOM_RESET_N: now also R218.1
- net GENADC_D6: now reaches J201.21 (P21)
- net GENADC_D7: now reaches J201.22 (P22)
- net GENADC_D8: now reaches J201.23 (P23)
- net GENADC_D9: now reaches J201.24 (P24)
- net GENADC_DCO: now reaches J201.25 (P25)
- net SYNC2_BIPHASE: now reaches J201.26 (P26)
- net HDMITX_D0: now reaches J201.32 (P32)
- net HDMITX_D1: now reaches J201.34 (P34)
- net HDMITX_D2: now reaches J201.36 (P36)
- net HDMITX_D3: now reaches J201.38 (P38)
- net HDMITX_D4: now reaches J201.41 (P41)
- net HDMITX_D5: now reaches J201.42 (P42)
- net HDMITX_D6: now reaches J201.43 (P43)
- net HDMITX_D7: now reaches J201.44 (P44)
- net HDMITX_D8: now reaches J201.45 (P45)
- net HDMITX_PCLK: now reaches J201.46 (P46)
- net HDMITX_D9: now reaches J201.47 (P47)
- net HDMITX_D10: now reaches J201.48 (P48)
- net HDMITX_D11: now reaches J201.51 (P51)
- net HDMITX_D12: now reaches J201.52 (P52)
- net HDMITX_D13: now reaches J201.53 (P53)
- net HDMITX_D14: now reaches J201.54 (P54)
- net HDMITX_D15: now reaches J201.55 (P55)
- net VIDOUT_CLKIN: now reaches J201.56 (P56)
- net HDMITX_DE: now reaches J201.57 (P57)
- net HDMITX_HS: now reaches J201.58 (P58)
- net HDMITX_VS: now reaches J201.61 (P61)
- net VIDOUT_P0: now reaches J201.62 (P62)
- net VIDOUT_P1: now reaches J201.63 (P63)
- net VIDOUT_P2: now reaches J201.64 (P64)
- net VIDOUT_P3: now reaches J201.65 (P65)
- net VIDOUT_P4: now reaches J201.66 (P66)
- net VIDOUT_P5: now reaches J201.67 (P67)
- net VIDOUT_P6: now reaches J201.68 (P68)
- net VIDOUT_P7: now reaches J201.71 (P71)
- net VIDOUT_P8: now reaches J201.72 (P72)
- net VIDOUT_P9: now reaches J201.73 (P73)
- net VIDOUT_P10: now reaches J201.74 (P74)
- net VIDOUT_P11: now reaches J201.75 (P75)
- net VIDOUT_P12: now reaches J201.76 (P76)
- net VIDOUT_P13: now reaches J201.77 (P77)
- net VIDOUT_P14: now reaches J201.78 (P78)
- net VIDOUT_P15: now reaches J201.81 (P81)
- net VIDOUT_HSYNC: now reaches J201.82 (P82)
- net VIDOUT_VSYNC: now reaches J201.83 (P83)
- net VIDOUT_SFL: now reaches J201.84 (P84)
- new net GND: C200.2, C201.2, C202.2, C203.2, C204.2, C205.2, C206.2, C207.2, C208.2, C209.2, C210.2, C211.2, C212.2, C213.2, R214.2, R217.2
- new net SOM_NOSEQ: J200.7 (P7), R214.1
