File: KiCad/SchindlerCarrierBoard_V1/SchindlerCarrierBoard_V1/05-analog-in.kicad_sch (KiCad schematic)
At the start: 32 parts, among them J500 73101-0120 (CVBS IN), J501 73101-0120 (comp Y IN), J502 73101-0120 (comp Pb IN), J503 73101-0120 (comp Pr IN), U500 ADV7280AWBCPZ-M-RL, Y500 28.63636MHz (ADV7280)

Commit message: Schindler 2.0: checkpoint — decoupling + functional audit, pre-edit save
Saves current carrier schematic state (all 12 sheets, KiCad re-saves) and
project docs before starting the decoupling/functional-fix wiring pass.

- docs/decoupling-audit.md: full per-chip decoupling audit (EXISTS /
  DATASHEET WANTS / PROPOSED ADDS) + "Functional fixes" section
  (COMP/PWRDWN*/VREG_VOUT floating, Y900 load caps; clocks verified
  present). ~91 proposed caps + ferrites; report-only, nothing placed.
- Other docs (bom-v1, refdes-map, spec, part-lock, etc.) synced.

No wiring changes — proposals await gate. Reference binaries (datasheet
JPGs/PDF, Manufacturing/) intentionally left untracked.

Co-Authored-By: Claude Opus 4.8 (1M context) <noreply@anthropic.com>
Parts:
- C500, C501, C502, C503, C504, C505, C506, C507, C508, C509, C510, C511: footprint (none) -> Capacitor_SMD:C_0805_2012Metric
- R500, R501, R502, R503, R504, R505, R506, R507: footprint (none) -> Resistor_SMD:R_0805_2012Metric
Changed lines of the file:
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@@
 			)
 		)
-		(property "Footprint" ""
+		(property "Footprint" "Capacitor_SMD:C_0805_2012Metric"
 			(at 400.05 95.25 0)
 			(hide yes)
@@
 			)
 		)
-		(property "Footprint" ""
+		(property "Footprint" "Capacitor_SMD:C_0805_2012Metric"
 			(at 279.4 204.47 0)
 			(hide yes)
@@
 			)
 		)
-		(property "Footprint" ""
+		(property "Footprint" "Resistor_SMD:R_0805_2012Metric"
 			(at 400.05 39.37 0)
 			(hide yes)
@@
 			)
 		)
-		(property "Footprint" ""
+		(property "Footprint" "Capacitor_SMD:C_0805_2012Metric"
 			(at 39.37 204.47 0)
 			(hide yes)
@@
 			)
 		)
-		(property "Footprint" ""
+		(property "Footprint" "Resistor_SMD:R_0805_2012Metric"
 			(at 400.05 149.86 0)
 			(hide yes)
@@
 			)
 		)
-		(property "Footprint" ""
+		(property "Footprint" "Resistor_SMD:R_0805_2012Metric"
 			(at 459.74 39.37 0)
 			(hide yes)
@@
 			)
 		)
-		(property "Footprint" ""
+		(property "Footprint" "Capacitor_SMD:C_0805_2012Metric"
 			(at 219.71 149.86 0)
 			(hide yes)
@@
 			)
 		)
-		(property "Footprint" ""
+		(property "Footprint" "Resistor_SMD:R_0805_2012Metric"
 			(at 279.4 95.25 0)
 			(hide yes)
@@
 			)
 		)
-		(property "Footprint" ""
+		(property "Footprint" "Resistor_SMD:R_0805_2012Metric"
 			(at 100.33 149.86 0)
 			(hide yes)
@@
 			)
 		)
-		(property "Footprint" ""
+		(property "Footprint" "Capacitor_SMD:C_0805_2012Metric"
 			(at 160.02 204.47 0)
 			(hide yes)
@@
 			)
 		)
-		(property "Footprint" ""
+		(property "Footprint" "Resistor_SMD:R_0805_2012Metric"
 			(at 39.37 149.86 0)
 			(hide yes)
@@
 			)
 		)
-		(property "Footprint" ""
+		(property "Footprint" "Capacitor_SMD:C_0805_2012Metric"
 			(at 459.74 149.86 0)
 			(hide yes)
@@
 			)
 		)
-		(property "Footprint" ""
+		(property "Footprint" "Capacitor_SMD:C_0805_2012Metric"
 			(at 39.37 95.25 0)
 			(hide yes)
@@
 			)
 		)
-		(property "Footprint" ""
+		(property "Footprint" "Capacitor_SMD:C_0805_2012Metric"
 			(at 340.36 204.47 0)
 			(hide yes)
@@
 			)
 		)
-		(property "Footprint" ""
+		(property "Footprint" "Capacitor_SMD:C_0805_2012Metric"
 			(at 340.36 95.25 0)
 			(hide yes)
@@
 			)
 		)
-		(property "Footprint" ""
+		(property "Footprint" "Capacitor_SMD:C_0805_2012Metric"
 			(at 100.33 95.25 0)
 			(hide yes)
@@
 			)
 		)
-		(property "Footprint" ""
+		(property "Footprint" "Capacitor_SMD:C_0805_2012Metric"
 			(at 160.02 149.86 0)
 			(hide yes)
@@
 			)
 		)
-		(property "Footprint" ""
+		(property "Footprint" "Resistor_SMD:R_0805_2012Metric"
 			(at 340.36 149.86 0)
 			(hide yes)
@@
 			)
 		)
-		(property "Footprint" ""
+		(property "Footprint" "Resistor_SMD:R_0805_2012Metric"
 			(at 219.71 95.25 0)
 			(hide yes)
@@
 			)
 		)
-		(property "Footprint" ""
+		(property "Footprint" "Capacitor_SMD:C_0805_2012Metric"
 			(at 219.71 204.47 0)
 			(hide yes)

Commit message: Schindler carrier: ADV7511 R_EXT/AVDD fix + symbol relabel; 116 PL nets wired; connector/riser decisions
- U403 ADV7511: add R406 (887R 1%) pin28 R_EXT->GND; wire pin29 AVDD->+1V8_A (match 34/41).
  Sheet-4 ERC pin_not_connected 2->0. Fixes missing TMDS bias ref + unpowered AVDD
  (would-not-work HDMI-out bug, caught pre-fab).
- JustinLibrary ADV7511KSTZ symbol relabel: pin2 SYNC->VSYNC, 28 EXT->R_EXT, 29 R_EXT->AVDD
  (cosmetic; connectivity is by pin number). [NOTE: JustinLibrary is unversioned/external — not in this repo; see report.]
- Pin-lock: 116 PL nets wired; ERC unconnected 899->668; schindler_plio.xdc + pin-lock-assignment.md.
- Connector domain + analog I/O riser decided (connector-domain.md); riser-mezzanine-plan.md rev2
  (gated proposal, not implemented).
- bom-v1 (R406), refdes-map (R406 + symbol-mislabel note), changelog.

Deferred to next commit (kept out so this push stays honest): eeschema Update Symbols from
Library on U403 (display refresh); netlist regen; HDMI +5V power_pin_not_driven x2 (J400/J401.18)
verification; riser stays gated.

Co-Authored-By: Claude Opus 4.8 (1M context) <noreply@anthropic.com>
Parts:
- added C512: 0.1uF (U500 DVDDIO), Capacitor_SMD:C_0805_2012Metric, symbol Device:C
- added C513, C514: 0.1uF (U500 DVDD), Capacitor_SMD:C_0805_2012Metric, symbol Device:C
- added C515: 0.1uF (U500 AVDD), Capacitor_SMD:C_0805_2012Metric, symbol Device:C
- added C516: 0.1uF (U500 PVDD), Capacitor_SMD:C_0805_2012Metric, symbol Device:C
- added C517: 10uF (U500 AVDD bulk), Capacitor_SMD:C_0805_2012Metric, symbol Device:C
- added R508: 10k (U500 PWRDWN* pull-up), symbol Device:R
Connections:
- net +1V8_D: now also C513.1, C514.1
- net +3V3: now also C512.1, R508.2
- net AVDD_DEC: now also C515.1, C516.1, C517.1
- net GND: now also C512.2, C513.2, C514.2, C515.2, C516.2, C517.2
- net IN0_AA: now also C500.1; no longer C500.2
- net IN0_BNC: now also C500.2; no longer C500.1
- net IN1_AA: now also R505.2; no longer R505.1
- net IN1_AIN: now also R505.1; no longer R505.2
- net ADV7280_P2: now reaches U500.10 (P2)
- net ADV7280_P1: now reaches U500.11 (P1)
- net ADV7280_P0: now reaches U500.12 (P0)
- net U500_PWRDWN_N: now reaches U500.31 (PWRDWN*)
- net U500_PWRDWN_N: now also R508.1
- net ADV7280_LLC: now reaches U500.32 (LCC)
- net ADV7280_P7: now reaches U500.5 (P7)
- net ADV7280_P6: now reaches U500.6 (P6)
- net ADV7280_P5: now reaches U500.7 (P5)
- net ADV7280_P4: now reaches U500.8 (P4)
- net ADV7280_P3: now reaches U500.9 (P3)
- no-connect marks 0 -> 3
Other:
- moved on the sheet: C500, C502, C503, C504, C505, C506, C507, C508, C509, C510, C511, D500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
