File: KiCad/SchindlerCarrierBoard_V1/SchindlerCarrierBoard_V1/08-genlock.kicad_sch (KiCad schematic)
At the start: 22 parts, among them J800 73101-0120 (REF IN, panel BNC), J801 73101-0120 (REF LOOP, panel B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, J802 Hirose U.FL-R-SMT-1 (REF IN c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, J803 Hirose U.FL-R-SMT-1 (REF LOOP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, U800 LTC6912CGN-2#PBF, U801 AD9204BCPZ-20, U802 TS5A23159 (REF 75R term sw, s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, U803 I2C GPIO expander (I2C_HK; te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

Commit message: Schindler 2.0: checkpoint — decoupling + functional audit, pre-edit save
Saves current carrier schematic state (all 12 sheets, KiCad re-saves) and
project docs before starting the decoupling/functional-fix wiring pass.

- docs/decoupling-audit.md: full per-chip decoupling audit (EXISTS /
  DATASHEET WANTS / PROPOSED ADDS) + "Functional fixes" section
  (COMP/PWRDWN*/VREG_VOUT floating, Y900 load caps; clocks verified
  present). ~91 proposed caps + ferrites; report-only, nothing placed.
- Other docs (bom-v1, refdes-map, spec, part-lock, etc.) synced.

No wiring changes — proposals await gate. Reference binaries (datasheet
JPGs/PDF, Manufacturing/) intentionally left untracked.

Co-Authored-By: Claude Opus 4.8 (1M context) <noreply@anthropic.com>
Parts:
- C800, C802, C803, C804, C805, C806, C807, C808: footprint (none) -> Capacitor_SMD:C_0805_2012Metric
- R800, R801, R802: footprint (none) -> Resistor_SMD:R_0805_2012Metric
Changed lines of the file:
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@@
 			)
 		)
-		(property "Footprint" ""
+		(property "Footprint" "Capacitor_SMD:C_0805_2012Metric"
 			(at 39.37 250.19 0)
 			(hide yes)
@@
 			)
 		)
-		(property "Footprint" ""
+		(property "Footprint" "Capacitor_SMD:C_0805_2012Metric"
 			(at 359.41 250.19 0)
 			(hide yes)
@@
 			)
 		)
-		(property "Footprint" ""
+		(property "Footprint" "Capacitor_SMD:C_0805_2012Metric"
 			(at 39.37 180.34 0)
 			(hide yes)
@@
 			)
 		)
-		(property "Footprint" ""
+		(property "Footprint" "Resistor_SMD:R_0805_2012Metric"
 			(at 279.4 180.34 0)
 			(hide yes)
@@
 			)
 		)
-		(property "Footprint" ""
+		(property "Footprint" "Capacitor_SMD:C_0805_2012Metric"
 			(at 199.39 250.19 0)
 			(hide yes)
@@
 			)
 		)
-		(property "Footprint" ""
+		(property "Footprint" "Capacitor_SMD:C_0805_2012Metric"
 			(at 199.39 180.34 0)
 			(hide yes)
@@
 			)
 		)
-		(property "Footprint" ""
+		(property "Footprint" "Resistor_SMD:R_0805_2012Metric"
 			(at 439.42 110.49 0)
 			(hide yes)
@@
 			)
 		)
-		(property "Footprint" ""
+		(property "Footprint" "Capacitor_SMD:C_0805_2012Metric"
 			(at 279.4 250.19 0)
 			(hide yes)
@@
 			)
 		)
-		(property "Footprint" ""
+		(property "Footprint" "Capacitor_SMD:C_0805_2012Metric"
 			(at 119.38 250.19 0)
 			(hide yes)
@@
 			)
 		)
-		(property "Footprint" ""
+		(property "Footprint" "Resistor_SMD:R_0805_2012Metric"
 			(at 359.41 180.34 0)
 			(hide yes)
@@
 			)
 		)
-		(property "Footprint" ""
+		(property "Footprint" "Capacitor_SMD:C_0805_2012Metric"
 			(at 439.42 180.34 0)
 			(hide yes)

Commit message: Schindler carrier: ADV7511 R_EXT/AVDD fix + symbol relabel; 116 PL nets wired; connector/riser decisions
- U403 ADV7511: add R406 (887R 1%) pin28 R_EXT->GND; wire pin29 AVDD->+1V8_A (match 34/41).
  Sheet-4 ERC pin_not_connected 2->0. Fixes missing TMDS bias ref + unpowered AVDD
  (would-not-work HDMI-out bug, caught pre-fab).
- JustinLibrary ADV7511KSTZ symbol relabel: pin2 SYNC->VSYNC, 28 EXT->R_EXT, 29 R_EXT->AVDD
  (cosmetic; connectivity is by pin number). [NOTE: JustinLibrary is unversioned/external — not in this repo; see report.]
- Pin-lock: 116 PL nets wired; ERC unconnected 899->668; schindler_plio.xdc + pin-lock-assignment.md.
- Connector domain + analog I/O riser decided (connector-domain.md); riser-mezzanine-plan.md rev2
  (gated proposal, not implemented).
- bom-v1 (R406), refdes-map (R406 + symbol-mislabel note), changelog.

Deferred to next commit (kept out so this push stays honest): eeschema Update Symbols from
Library on U403 (display refresh); netlist regen; HDMI +5V power_pin_not_driven x2 (J400/J401.18)
verification; riser stays gated.

Co-Authored-By: Claude Opus 4.8 (1M context) <noreply@anthropic.com>
Parts:
- removed J800: 73101-0120 (REF IN, panel BNC), symbol Connector:Conn_Coaxial
- removed J801: 73101-0120 (REF LOOP, panel BNC), symbol Connector:Conn_Coaxial
- added C809, C810, C811, C812, C813, C814, C815: 0.1uF (U801 AVDD), symbol Device:C
- added C816, C817, C818: 0.1uF (U801 DRVDD), symbol Device:C
- added C819: 10uF (U801 AVDD bulk), symbol Device:C
- added C820: 1uF (U800 V+), symbol Device:C
Connections:
- net +1V8_D: now also C816.1, C817.1, C818.1
- net +5V_PGA: now also C820.1
- net AVDD_GENADC: now also C809.1, C810.1, C811.1, C812.1, C813.1, C814.1, C815.1, C819.1
- net GND: now also C809.2, C810.2, C811.2, C812.2, C813.2, C814.2, C815.2, C816.2, C817.2, C818.2, C819.2, C820.2
- net GENADC_DCO: now reaches U801.24 (DCOA)
- net GENADC_D0: now reaches U801.32 (D0A(LSB))
- net GENADC_D1: now reaches U801.33 (D1A)
- net GENADC_D2: now reaches U801.34 (D2A)
- net GENADC_D3: now reaches U801.35 (D3A)
- net GENADC_D4: now reaches U801.36 (D4A)
- net GENADC_D5: now reaches U801.38 (D5A)
- net GENADC_D6: now reaches U801.39 (D6A)
- net GENADC_D7: now reaches U801.40 (D7A)
- net GENADC_D8: now reaches U801.41 (D8A)
- net GENADC_D9: now reaches U801.42 (D9A(MSB))
Other:
- note added: "SYNC IN (J802) / SYNC LOOP (J803): carrier U.FL landing. Panel BNC + 75R pigtail (Option A) = chassis BOM, NOT carrier PCB. See panel-layout.md / 01-spec 3.7."
- moved on the sheet: C800, C802, C803, C804, C805, C806, C807, C808, D800A, D800B, D801, D802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
