File: KiCad/SchindlerCarrierBoard_V1/SchindlerCarrierBoard_V1/09-clock-sync.kicad_sch (KiCad schematic)
At the start: 27 parts, among them J900 73101-0120 (SYNC OUT 1), J901 73101-0120 (SYNC OUT 2), J902 RP2040 SWD hdr, U900 RP2040 (genlock MCU), U901 W25Q128JVSIQ, U902 Si5351A-B-GTR, U903 AD9742 (SYNC1 DAC), U904 LMH6643MAX/NOPB (sync drivers), Y900 12MHz, Y901 25MHz

Commit message: Schindler 2.0: checkpoint — decoupling + functional audit, pre-edit save
Saves current carrier schematic state (all 12 sheets, KiCad re-saves) and
project docs before starting the decoupling/functional-fix wiring pass.

- docs/decoupling-audit.md: full per-chip decoupling audit (EXISTS /
  DATASHEET WANTS / PROPOSED ADDS) + "Functional fixes" section
  (COMP/PWRDWN*/VREG_VOUT floating, Y900 load caps; clocks verified
  present). ~91 proposed caps + ferrites; report-only, nothing placed.
- Other docs (bom-v1, refdes-map, spec, part-lock, etc.) synced.

No wiring changes — proposals await gate. Reference binaries (datasheet
JPGs/PDF, Manufacturing/) intentionally left untracked.

Co-Authored-By: Claude Opus 4.8 (1M context) <noreply@anthropic.com>
Parts:
- C900, C901, C902, C903, C904: footprint (none) -> Capacitor_SMD:C_0805_2012Metric
- R900, R901, R902, R903, R904, R905, R906, R907, R908, R909: footprint (none) -> Resistor_SMD:R_0805_2012Metric
Other:
- moved on the sheet: C900, C901, C902, C903, C904, D900, D901, J900, J901, J902, R900, R901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

Commit message: Schindler carrier: ADV7511 R_EXT/AVDD fix + symbol relabel; 116 PL nets wired; connector/riser decisions
- U403 ADV7511: add R406 (887R 1%) pin28 R_EXT->GND; wire pin29 AVDD->+1V8_A (match 34/41).
  Sheet-4 ERC pin_not_connected 2->0. Fixes missing TMDS bias ref + unpowered AVDD
  (would-not-work HDMI-out bug, caught pre-fab).
- JustinLibrary ADV7511KSTZ symbol relabel: pin2 SYNC->VSYNC, 28 EXT->R_EXT, 29 R_EXT->AVDD
  (cosmetic; connectivity is by pin number). [NOTE: JustinLibrary is unversioned/external — not in this repo; see report.]
- Pin-lock: 116 PL nets wired; ERC unconnected 899->668; schindler_plio.xdc + pin-lock-assignment.md.
- Connector domain + analog I/O riser decided (connector-domain.md); riser-mezzanine-plan.md rev2
  (gated proposal, not implemented).
- bom-v1 (R406), refdes-map (R406 + symbol-mislabel note), changelog.

Deferred to next commit (kept out so this push stays honest): eeschema Update Symbols from
Library on U403 (display refresh); netlist regen; HDMI +5V power_pin_not_driven x2 (J400/J401.18)
verification; riser stays gated.

Co-Authored-By: Claude Opus 4.8 (1M context) <noreply@anthropic.com>
Parts:
- added C905: 15pF (Y900 XIN load, DNP-verify CL), symbol Device:C
- added C906: 15pF (Y900 XOUT load, DNP-verify CL), symbol Device:C
- added C907, C908, C909, C910, C911, C912: 0.1uF (U900 IOVDD), symbol Device:C
- added C913: 1uF (U900 VREG_VOUT), symbol Device:C
- added C914, C916: 0.1uF (U900 DVDD), symbol Device:C
- added C917: 0.1uF (U900 USB_VDD), symbol Device:C
- added C918: 4.7uF (U900 IOVDD bulk), symbol Device:C
- added C919: 0.1uF (U901 VCC), symbol Device:C
- added C920: 0.1uF (U902 VDD), symbol Device:C
- added C921: 1uF (U902 VDD bulk), symbol Device:C
- added C922: 0.1uF (U902 VDDO), symbol Device:C
- added C923: 0.1uF (U903 AVDD), symbol Device:C
- added C924: 0.1uF (U903 DVDD), symbol Device:C
- added C925: 10uF (U903 AVDD/DVDD bulk), symbol Device:C
Connections:
- net +3V3: now also C907.1, C908.1, C909.1, C910.1, C911.1, C912.1, C917.1, C918.1, C919.1, C920.1, C921.1, C922.1, C923.1, C924.1, C925.1
- net GENLK_XI: now also C905.1
- net GENLK_XO: now also C906.1
- net GND: now also C905.2, C906.2, C907.2, C908.2, C909.2, C910.2, C911.2, C912.2, C913.2, C914.2, C916.2, C917.2, C918.2, C919.2, C920.2, C921.2, C922.2, C923.2, C924.2, C925.2
- net RP2040_VCORE: now also C913.1, C914.1, C916.1
- net SYNC1_DAC_DB11: now reaches U903.1 ((MSB)DB11)
- net SYNC1_DAC_DB2: now reaches U903.10 (DB2)
- net SYNC1_DAC_DB1: now reaches U903.11 (DB1)
- net SYNC1_DAC_DB0: now reaches U903.12 ((LSB)DB0)
- net SYNC1_DAC_DB10: now reaches U903.2 (DB10)
- net SYNC1_DAC_CLK: now reaches U903.28 (CLOCK)
- net SYNC1_DAC_DB9: now reaches U903.3 (DB9)
- net SYNC1_DAC_DB8: now reaches U903.4 (DB8)
- net SYNC1_DAC_DB7: now reaches U903.5 (DB7)
- net SYNC1_DAC_DB6: now reaches U903.6 (DB6)
- net SYNC1_DAC_DB5: now reaches U903.7 (DB5)
- net SYNC1_DAC_DB4: now reaches U903.8 (DB4)
- net SYNC1_DAC_DB3: now reaches U903.9 (DB3)
- net SYNC2_LTC_IN renamed SYNC2_BIPHASE
Other:
- note added: "Si5351 (U902): no external XTAL load caps; firmware sets XTAL_CL to match Y901."
- moved on the sheet: C904
