File: KiCad/SchindlerCarrierBoard_V1/SchindlerCarrierBoard_V1/10-control-net.kicad_sch (KiCad schematic)
At the start: 4 parts, among them J1000 JXD1-0001NL, J1001 USB4085-GF-A, J1002 CONREVSMA001 RP-SMA (ESP32-S3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, U1001 TPD4S014DBVR

Commit message: Schindler carrier: ADV7511 R_EXT/AVDD fix + symbol relabel; 116 PL nets wired; connector/riser decisions
- U403 ADV7511: add R406 (887R 1%) pin28 R_EXT->GND; wire pin29 AVDD->+1V8_A (match 34/41).
  Sheet-4 ERC pin_not_connected 2->0. Fixes missing TMDS bias ref + unpowered AVDD
  (would-not-work HDMI-out bug, caught pre-fab).
- JustinLibrary ADV7511KSTZ symbol relabel: pin2 SYNC->VSYNC, 28 EXT->R_EXT, 29 R_EXT->AVDD
  (cosmetic; connectivity is by pin number). [NOTE: JustinLibrary is unversioned/external — not in this repo; see report.]
- Pin-lock: 116 PL nets wired; ERC unconnected 899->668; schindler_plio.xdc + pin-lock-assignment.md.
- Connector domain + analog I/O riser decided (connector-domain.md); riser-mezzanine-plan.md rev2
  (gated proposal, not implemented).
- bom-v1 (R406), refdes-map (R406 + symbol-mislabel note), changelog.

Deferred to next commit (kept out so this push stays honest): eeschema Update Symbols from
Library on U403 (display refresh); netlist regen; HDMI +5V power_pin_not_driven x2 (J400/J401.18)
verification; riser stays gated.

Co-Authored-By: Claude Opus 4.8 (1M context) <noreply@anthropic.com>
Other:
- moved on the sheet: J1000, J1001, J1002, U1001
Changed lines of the file:
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@@
 	(global_label "+5V"
 		(shape input)
-		(at 177.8 22.86 0)
-		(effects
-			(font
-				(size 1.27 1.27)
-			)
-			(justify left)
-		)
-		(property "Intersheetrefs" "${INTERSHEET_REFS}"
-			(at 177.8 22.86 0)
+		(at 349.25 213.36 180)
+		(effects
+			(font
+				(size 1.27 1.27)
+			)
+			(justify right)
+		)
+		(property "Intersheetrefs" "${INTERSHEET_REFS}"
+			(at 349.25 213.36 0)
 			(hide yes)
 			(show_name no)
@@
 	(global_label "GND"
 		(shape input)
-		(at 110.49 53.34 0)
-		(effects
-			(font
-				(size 1.27 1.27)
-			)
-			(justify left)
-		)
-		(property "Intersheetrefs" "${INTERSHEET_REFS}"
-			(at 110.49 53.34 0)
+		(at 281.94 243.84 270)
+		(effects
+			(font
+				(size 1.27 1.27)
+			)
+			(justify right)
+		)
+		(property "Intersheetrefs" "${INTERSHEET_REFS}"
+			(at 281.94 243.84 90)
 			(hide yes)
 			(show_name no)
@@
 	(global_label "GND"
 		(shape input)
-		(at 190.5 43.18 0)
-		(effects
-			(font
-				(size 1.27 1.27)
-			)
-			(justify left)
-		)
-		(property "Intersheetrefs" "${INTERSHEET_REFS}"
-			(at 190.5 43.18 0)
+		(at 361.95 233.68 270)
+		(effects
+			(font
+				(size 1.27 1.27)
+			)
+			(justify right)
+		)
+		(property "Intersheetrefs" "${INTERSHEET_REFS}"
+			(at 361.95 233.68 90)
+			(hide yes)
+			(show_name no)
+			(do_not_autoplace no)
+			(effects
+				(font
+					(size 1.27 1.27)
+				)
+			)
+		)
+	)
+	(global_label "ESP_ANT"
+		(shape input)
+		(at 436.88 220.98 180)
+		(effects
+			(font
+				(size 1.27 1.27)
+			)
+			(justify right)
+		)
+		(property "Intersheetrefs" "${INTERSHEET_REFS}"
+			(at 436.88 220.98 0)
 			(hide yes)
 			(show_name no)
@@
 	(global_label "GND"
 		(shape input)
-		(at 110.49 53.34 0)
-		(effects
-			(font
-				(size 1.27 1.27)
-			)
-			(justify left)
-		)
-		(property "Intersheetrefs" "${INTERSHEET_REFS}"
-			(at 110.49 53.34 0)
+		(at 441.96 226.06 270)
+		(effects
+			(font
+				(size 1.27 1.27)
+			)
+			(justify right)
+		)
+		(property "Intersheetrefs" "${INTERSHEET_REFS}"
+			(at 441.96 226.06 90)
 			(hide yes)
 			(show_name no)
@@
 	(global_label "GND"
 		(shape input)
-		(at 110.49 53.34 0)
-		(effects
-			(font
-				(size 1.27 1.27)
-			)
-			(justify left)
-		)
-		(property "Intersheetrefs" "${INTERSHEET_REFS}"
-			(at 110.49 53.34 0)
-			(hide yes)
-			(show_name no)
-			(do_not_autoplace no)
-			(effects
-				(font
-					(size 1.27 1.27)
-				)
-			)
-		)
-	)
-	(global_label "ESP_ANT"
-		(shape input)
-		(at 265.43 30.48 0)
-		(effects
-			(font
-				(size 1.27 1.27)
-			)
-			(justify left)
-		)
-		(property "Intersheetrefs" "${INTERSHEET_REFS}"
-			(at 265.43 30.48 0)
-			(hide yes)
-			(show_name no)
-			(do_not_autoplace no)
-			(effects
-				(font
-					(size 1.27 1.27)
-				)
-			)
-		)
-	)
-	(global_label "+5V"
-		(shape input)
-		(at 177.8 22.86 0)
-		(effects
-			(font
-				(size 1.27 1.27)
-			)
-			(justify left)
-		)
-		(property "Intersheetrefs" "${INTERSHEET_REFS}"
-			(at 177.8 22.86 0)
-			(hide yes)
-			(show_name no)
-			(do_not_autoplace no)
-			(effects
-				(font
-					(size 1.27 1.27)
-				)
-			)
-		)
-	)
-	(global_label "GND"
-		(shape input)
-		(at 110.49 53.34 0)
-		(effects
-			(font
-				(size 1.27 1.27)
-			)
-			(justify left)
-		)
-		(property "Intersheetrefs" "${INTERSHEET_REFS}"
-			(at 110.49 53.34 0)
-			(hide yes)
-			(show_name no)
-			(do_not_autoplace no)
-			(effects
-				(font
-					(size 1.27 1.27)
-				)
-			)
-		)
-	)
-	(global_label "GND"
-		(shape input)
-		(at 270.51 35.56 0)
-		(effects
-			(font
-				(size 1.27 1.27)
-			)
-			(justify left)
-		)
-		(property "Intersheetrefs" "${INTERSHEET_REFS}"
-			(at 270.51 35.56 0)
-			(hide yes)
-			(show_name no)
-			(do_not_autoplace no)
-			(effects
-				(font
-					(size 1.27 1.27)
-				)
-			)
-		)
-	)
-	(global_label "GND"
-		(shape input)
-		(at 193.04 43.18 0)
-		(effects
-			(font
-				(size 1.27 1.27)
-			)
-			(justify left)
-		)
-		(property "Intersheetrefs" "${INTERSHEET_REFS}"
-			(at 193.04 43.18 0)
+		(at 364.49 233.68 270)
+		(effects
+			(font
+				(size 1.27 1.27)
+			)
+			(justify right)
+		)
+		(property "Intersheetrefs" "${INTERSHEET_REFS}"
+			(at 364.49 233.68 90)
 			(hide yes)
 			(show_name no)
@@
 	(symbol
 		(lib_id "Power_Protection:TPD4S014")
-		(at 190.5 30.48 0)
+		(at 361.95 220.98 0)
 		(unit 1)
 		(body_style 1)
@@
 		(dnp no)
 		(property "Reference" "U1001"
-			(at 196.85 27.94 0)
+			(at 359.664 209.296 0)
 			(show_name no)
 			(do_not_autoplace no)
@@
 		)
 		(property "Value" "TPD4S014DBVR"
-			(at 196.85 33.02 0)
+			(at 366.268 232.918 0)
 			(show_name no)
 			(do_not_autoplace no)
@@
 		)
 		(property "Footprint" ""
-			(at 190.5 30.48 0)
+			(at 361.95 220.98 0)
 			(hide yes)
 			(show_name no)
@@
 		)
 		(property "Datasheet" ""
-			(at 190.5 30.48 0)
+			(at 361.95 220.98 0)
 			(show_name no)
 			(do_not_autoplace no)
@@
 		)
 		(property "Description" ""
-			(at 190.5 30.48 0)
+			(at 361.95 220.98 0)
 			(show_name no)
 			(do_not_autoplace no)
@@
 	(symbol
 		(lib_id "Connector:USB_C_Receptacle_USB2.0_16P")
-		(at 110.49 30.48 0)
+		(at 281.94 220.98 0)
 		(unit 1)
 		(body_style 1)
@@
 		(dnp no)
 		(property "Reference" "J1001"
-			(at 116.84 27.94 0)
+			(at 279.654 201.93 0)
 			(show_name no)
 			(do_not_autoplace no)
@@
 		)
 		(property "Value" "USB4085-GF-A"
-			(at 116.84 33.02 0)
+			(at 285.242 240.538 0)
 			(show_name no)
 			(do_not_autoplace no)
@@
 		)
 		(property "Footprint" ""
-			(at 110.49 30.48 0)
+			(at 281.94 220.98 0)
 			(hide yes)
 			(show_name no)
@@
 		)
 		(property "Datasheet" ""
-			(at 110.49 30.48 0)
+			(at 281.94 220.98 0)
 			(show_name no)
 			(do_not_autoplace no)
@@
 		)
 		(property "Description" ""
-			(at 110.49 30.48 0)
+			(at 281.94 220.98 0)
 			(show_name no)
 			(do_not_autoplace no)
@@
 	(symbol
 		(lib_id "Connector:Conn_Coaxial")
-		(at 270.51 30.48 0)
+		(at 441.96 220.98 0)
 		(unit 1)
 		(body_style 1)
@@
 		(dnp no)
 		(property "Reference" "J1002"
-			(at 276.86 27.94 0)
+			(at 448.31 218.44 0)
 			(show_name no)
 			(do_not_autoplace no)
@@
 		)
 		(property "Value" "CONREVSMA001 RP-SMA (ESP32-S3 WiFi ant: A2 U.FL->coax->J1002)"
-			(at 276.86 33.02 0)
+			(at 448.31 223.52 0)
 			(show_name no)
 			(do_not_autoplace no)
@@
 		)
 		(property "Footprint" ""
-			(at 270.51 30.48 0)
+			(at 441.96 220.98 0)
 			(hide yes)
 			(show_name no)
@@
 		)
 		(property "Datasheet" ""
-			(at 270.51 30.48 0)
+			(at 441.96 220.98 0)
 			(show_name no)
 			(do_not_autoplace no)
@@
 		)
 		(property "Description" ""
-			(at 270.51 30.48 0)
+			(at 441.96 220.98 0)
 			(show_name no)
 			(do_not_autoplace no)
@@
 	(symbol
 		(lib_id "Connector:RJ45")
-		(at 30.48 30.48 0)
+		(at 201.93 220.98 0)
 		(unit 1)
 		(body_style 1)
@@
 		(dnp no)
 		(property "Reference" "J1000"
-			(at 36.83 27.94 0)
+			(at 199.644 207.01 0)
 			(show_name no)
 			(do_not_autoplace no)
@@
 		)
 		(property "Value" "JXD1-0001NL"
-			(at 36.83 33.02 0)
+			(at 195.072 232.918 0)
 			(show_name no)
 			(do_not_autoplace no)
@@
 		)
 		(property "Footprint" ""
-			(at 30.48 30.48 0)
+			(at 201.93 220.98 0)
 			(hide yes)
 			(show_name no)
@@
 		)
 		(property "Datasheet" ""
-			(at 30.48 30.48 0)
+			(at 201.93 220.98 0)
 			(show_name no)
 			(do_not_autoplace no)
@@
 		)
 		(property "Description" ""
-			(at 30.48 30.48 0)
-			(show_name no)
-			(do_not_autoplace no)
+			(at 201.93 220.98 0)
+			(show_name no)
+			(do_not_autoplace no)
