File: KiCad/SchindlerCarrierBoard_V1/SchindlerCarrierBoard_V1/SchindlerCarrierBoard_V1.kicad_sch (KiCad schematic)
At the start: 11 parts

Commit message: Schindler 2.0: checkpoint — decoupling + functional audit, pre-edit save
Saves current carrier schematic state (all 12 sheets, KiCad re-saves) and
project docs before starting the decoupling/functional-fix wiring pass.

- docs/decoupling-audit.md: full per-chip decoupling audit (EXISTS /
  DATASHEET WANTS / PROPOSED ADDS) + "Functional fixes" section
  (COMP/PWRDWN*/VREG_VOUT floating, Y900 load caps; clocks verified
  present). ~91 proposed caps + ferrites; report-only, nothing placed.
- Other docs (bom-v1, refdes-map, spec, part-lock, etc.) synced.

No wiring changes — proposals await gate. Reference binaries (datasheet
JPGs/PDF, Manufacturing/) intentionally left untracked.

Co-Authored-By: Claude Opus 4.8 (1M context) <noreply@anthropic.com>
Parts:
- MP101, MP102, MP103, MP104, MP105, MP106, MP107, MP108: footprint (none) -> MountingHole:MountingHole_3.2mm_M3
Changed lines of the file:
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@@
 			)
 		)
-		(property "Footprint" ""
+		(property "Footprint" "MountingHole:MountingHole_3.2mm_M3"
 			(at 190.5 250.19 0)
+			(hide yes)
 			(show_name no)
 			(do_not_autoplace no)
@@
 			)
 		)
-		(property "Footprint" ""
+		(property "Footprint" "MountingHole:MountingHole_3.2mm_M3"
 			(at 69.85 265.43 0)
+			(hide yes)
 			(show_name no)
 			(do_not_autoplace no)
@@
 			)
 		)
-		(property "Footprint" ""
+		(property "Footprint" "MountingHole:MountingHole_3.2mm_M3"
 			(at 110.49 250.19 0)
+			(hide yes)
 			(show_name no)
 			(do_not_autoplace no)
@@
 			)
 		)
-		(property "Footprint" ""
+		(property "Footprint" "MountingHole:MountingHole_3.2mm_M3"
 			(at 30.48 265.43 0)
+			(hide yes)
 			(show_name no)
 			(do_not_autoplace no)
@@
 		(property "Footprint" ""
 			(at 149.86 265.43 0)
+			(hide yes)
 			(show_name no)
 			(do_not_autoplace no)
@@
 			)
 		)
-		(property "Footprint" ""
+		(property "Footprint" "MountingHole:MountingHole_3.2mm_M3"
 			(at 30.48 250.19 0)
+			(hide yes)
 			(show_name no)
 			(do_not_autoplace no)
@@
 			)
 		)
-		(property "Footprint" ""
+		(property "Footprint" "MountingHole:MountingHole_3.2mm_M3"
 			(at 229.87 250.19 0)
+			(hide yes)
 			(show_name no)
 			(do_not_autoplace no)
@@
 		(property "Footprint" ""
 			(at 110.49 265.43 0)
+			(hide yes)
 			(show_name no)
 			(do_not_autoplace no)
@@
 			)
 		)
-		(property "Footprint" ""
+		(property "Footprint" "MountingHole:MountingHole_3.2mm_M3"
 			(at 69.85 250.19 0)
+			(hide yes)
 			(show_name no)
 			(do_not_autoplace no)
@@
 		(property "Footprint" ""
 			(at 190.5 265.43 0)
+			(hide yes)
 			(show_name no)
 			(do_not_autoplace no)
@@
 			)
 		)
-		(property "Footprint" ""
+		(property "Footprint" "MountingHole:MountingHole_3.2mm_M3"
 			(at 149.86 250.19 0)
-			(show_name no)
-			(do_not_autoplace no)
+			(hide yes)
+			(show_name no)
+			(do_not_autoplace no)
